File: kicad_source/History.sch (KiCad schematic (older format))
At the start: 0 parts

Commit message: added values in schematic, generated pdf schematic
Other:
- note added: "1.0"
- note added: "2019-12-29"
- note added: "Bernhard Mayer"
- note added: "initial release"
Changed lines of the file:
@@
 EESchema Schematic File Version 4
-LIBS:HighPowerMotorFeatherWing-cache
-EELAYER 26 0
+EELAYER 30 0
 EELAYER END
 $Descr A4 11693 8268
@@
 Sheet 5 5
 Title ""
-Date ""
+Date "2019-12-29"
 Rev ""
 Comp ""
@@
 Comment4 ""
 $EndDescr
+Text Notes 850  900  0    60   ~ 0
+1.0
+Text Notes 1350 900  0    60   ~ 0
+2019-12-29
+Text Notes 2300 900  0    60   ~ 0
+Bernhard Mayer
+Text Notes 3350 900  0    60   ~ 0
+initial release
 $EndSCHEMATC
